File: hardware/LIONv3/POWER.kicad_sch (KiCad schematic)
At the start: 28 parts, among them U10 INA226AIDGSR, U11 TPS259474ARPWR, U12 XL-1608UGC-04, U13 XL-1608SURC-06, U16 HC-1_25-2PWT, U17 HC-1_25-2PWT, U18 HC-1_25-2PWT, U20 TLV76733DRVR

Commit message: feat(hardware): add TestPoints
Parts:
- added TP10, TP11, TP12: TestPoint_Square, TestPoint:TestPoint_Pad_D1.5mm, symbol Connector:TestPoint_Square
- renumbered C20 to C13, C17 to C14, C6 to C15, C21 to C16, C18 to C17, C19 to C18, C16 to C19, D7 to D4, D6 to D5, R19 to R18, R22 to R19, R24 to R20, R20 to R21, R23 to R22, R32 to R23, R25 to R24, R21 to R25, R18 to R26, R17 to R27, U12 to U13, U11 to U14, U20 to U15, U13 to U16, U10 to U17, U17 to U18, U16 to U19, U18 to U20
Connections:
- net +3.3V: now also TP10.1
- net +3.3V_LDO: now also TP11.1
- net LED_FAULT: now also TP12.1
Other:
- note added: "YLRY06-1-50F"
- moved on the sheet: C19

Commit message: feat(hardware): start PCB design
Parts:
- C13, C14: footprint Capacitor_SMD:C_0402_1005Metric -> Capacitor_SMD:C_0603_1608Metric
Changed lines of the file:
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@@
 			)
 		)
-		(property "Footprint" "Capacitor_SMD:C_0402_1005Metric"
+		(property "Footprint" "Capacitor_SMD:C_0603_1608Metric"
 			(at 116.84 41.91 0)
 			(hide yes)
@@
 			)
 		)
-		(property "Footprint" "Capacitor_SMD:C_0402_1005Metric"
+		(property "Footprint" "Capacitor_SMD:C_0603_1608Metric"
 			(at 203.2 35.56 0)
 			(hide yes)
