File: hardware/LIONv3/LIONv3.kicad_sch (KiCad schematic)
At the start: 40 parts, among them SW1 RESET, SW2 BOOT, U1 HC-1_25-2PWT, U2 HC-1_25-2PWT, U3 ESP32-C6-MINI-1-N4, U5 HC-1_25-2PWT, U6 TMP112AIDRLR, U7 USBLC6-2SC6, U8 TYPE-C_16PIN_2MD(073)

Commit message: feat(hardware): finish PDN
Connections:
- net D+: now also U7.3 (I/O2); no longer U7.1 (I/O1)
- net D-: now also U7.1 (I/O1); no longer U7.3 (I/O2)
- net USB_D+: now also U7.4 (I/O2); no longer U7.6 (I/O1)
- net USB_D-: now also U7.6 (I/O1); no longer U7.4 (I/O2)
