File: hardware/LIONv3/LIONv3.kicad_pcb (KiCad board)
At the start: 4 copper layers, 50.1 x 85.2 mm, 85 parts, among them SW1 RESET, SW2 BOOT, U1 HC-1_25-2PWT, U10 E80-900M2213S, U11 W25Q16JVSSIQTR, U12 XL-1608UBC-04, U13 XL-1608UGC-04, U14 TPS259474ARPWR, U15 TLV76733DRVR, U16 XL-1608SURC-06, U17 INA226AIDGSR, U18 HC-1_25-2PWT, U19 HC-1_25-2PWT, U2 HC-1_25-2PWT, U20 HC-1_25-2PWT, U21 TCAN3414DR, U3 ESP32-C6-MINI-1-N4, U5 HC-1_25-2PWT, U6 TMP112AIDRLR, U7 USBLC6-2SC6, U8 TYPE-C_16PIN_2MD(073), U9 INA226AIDGSR

Commit message: feat(hardware): finish main routing
Parts:
- added REF**: OSHW-Logo_5.7x6mm_SilkScreen, Symbol:OSHW-Logo_5.7x6mm_SilkScreen, F.Cu at (354.9, 69.5)
- C20, C21: moved to B.Cu
- moved R20 49.4 mm to (332.6, 86.3), turned to 0 degrees
- moved R24 49.3 mm to (332.6, 89.2), turned to 0 degrees
- moved R17 49.2 mm to (332.6, 92.0), turned to 0 degrees
- moved U13 48.9 mm to (332.9, 87.8), turned to 180 degrees
- moved U16 48.9 mm to (332.8, 90.6), turned to 180 degrees
- moved U12 48.8 mm to (332.8, 93.4), turned to 180 degrees
- moved C20 29.9 mm to (348.4, 70.8), turned to -90 degrees
- moved C21 21.5 mm to (350.1, 70.8), turned to -90 degrees
- moved D1 2.78 mm to (321.7, 76.3)
- moved C3 1.05 mm to (322.1, 75.0), turned to 0 degrees
- moved R4 0.91 mm to (334.6, 74.8)
- moved SW2 0.71 mm to (334.5, 78.6), turned to 180 degrees
- moved D2 0.70 mm to (334.5, 76.3)
- moved JP1 0.69 mm to (360.1, 62.3)
- moved C22 0.55 mm to (359.6, 60.4), turned to 0 degrees
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Connections:
- R11 pad 1: 3.3V_RF -> +3.3V
- U5 pad 1: /I2C_SCL -> /I2C_SDA
- U5 pad 2: /I2C_SDA -> /I2C_SCL
Routing:
- net /I2C_SDA: track 19.3 -> 66.0 mm, vias 1 -> 5
- net /I2C_SCL: track 17.2 -> 63.3 mm, vias 3 -> 5
- net /CAN_STB: track 0.00 -> 33.1 mm, vias 0 -> 1
- net /CAN_RX: track 0.00 -> 27.7 mm, vias 0 -> 1
- net /LR_LED: track 0.00 -> 23.2 mm, vias 0 -> 2
- net /FLASH_CS#: track 1.94 -> 25.0 mm, vias 0 -> 2
- net /TMP_ALERT: track 14.1 -> 34.7 mm, vias 1 -> 2
- net /CAN_TX: track 0.00 -> 20.5 mm, vias 0 -> 1
- net /POWER/LED_FAULT: track 0.98 -> 14.3 mm
- net +3.3V_eFuse: track 4.10 -> 12.0 mm, vias 0 -> 1
- net +3.3V: track 14.2 -> 20.6 mm, vias 29 -> 32
- net +3.3V_LDO: track 6.68 -> 9.62 mm, vias 1 -> 0
- net GND: track 11.3 -> 13.7 mm, vias 381 -> 383
- net Net-(D1-A2): track 14.0 -> 11.9 mm
- net /INA_ALERT: track 32.9 -> 31.2 mm
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Other:
- board text added: "CANbus"

Commit message: feat(hardware): complete 90% of PCB layout, final tweaks remaining
Parts:
- added G***: LOGO, LOGO, F.Cu at (362.2, 68.6)
- added G***: LOGO, LOGO, B.Cu at (335.6, 71.7)
- added G***: LOGO, LOGO, B.Cu at (341.0, 120.2)
- moved REF** 0.50 mm to (355.4, 69.4)
Other:
- board text added: "+3.3V"
- board text added: "+5V"
- board text added: "By: Rodrigo A."
- board text added: "GND"
- board text added: "I2C"
- board text added: "RX"
- board text added: "TX"
- board text added: "UART"
- board text added: "v1•e8e3db53"
- board text removed: "LIONv3-R"
